Commit message: Add URDF and OBJ files for Livox Lidar display model
- Created livox_display.urdf.xacro to define the visual representation of the Livox Lidar sensor, including a dynamic sensor frame and a visual-only mesh.
- Added robot_base_cone.obj to represent the base of the sensor as a 16-sided cone with specified dimensions and centered at the origin.

File: src/livox_lidar_example/worlds/livox_example.world.xacro (robot description, xacro)
@@ -9,4 +9,7 @@
   <xacro:include filename="$(find livox_lidar_gz_sensor)/urdf/livox_mid40.xacro"/>
   <xacro:include filename="$(find livox_lidar_gz_sensor)/urdf/livox_horizon.xacro"/>
+  <xacro:include filename="$(find livox_lidar_gz_sensor)/urdf/livox_avia.xacro"/>
+  <xacro:include filename="$(find livox_lidar_gz_sensor)/urdf/livox_HAP.xacro"/>
+  <xacro:include filename="$(find livox_lidar_gz_sensor)/urdf/livox_tele.xacro"/>
   <world name="livox_example">
     <!-- Keep movable objects suspended while allowing GUI pose commands. -->
@@ -46,9 +49,10 @@
       <link name="ground_link">
         <collision name="ground_collision">
-          <geometry>
-            <plane>
-              <normal>0 0 1</normal>
-              <size>20 20</size>
-            </plane>
+          <pose>0 0 -0.05 0 0 0</pose>
+          <geometry>
+            <!-- Keep the physics surface bounded like the visible floor.
+                 An SDF plane is infinite and creates very distant returns
+                 for rays only slightly below the horizon. -->
+            <box><size>20 20 0.1</size></box>
           </geometry>
         </collision>
@@ -187,5 +191,7 @@
         </collision>
       </link>
-      <xacro:livox_horizon_link
+      <!-- Keep the sensor body above the cone tip; the example uses a
+           noise-free cloud so ground-plane geometry is easy to inspect. -->
+      <xacro:livox_mid360_link
         link_name="livox_left"
         link_pose="0 0 0.6 0 0 0"
@@ -236,5 +242,5 @@
         </collision>
       </link>
-      <xacro:livox_mid360_link
+      <xacro:livox_avia_link
         link_name="livox_right"
         link_pose="0 0 0.6 0 0 0"

File: src/livox_lidar_gz_sensor/urdf/livox_HAP.xacro (robot description, xacro)
@@ -17,5 +17,5 @@
       downsample:=1
       noise_mean:=0.0
-      noise_stddev:=0.01">
+      noise_stddev:=0.0">
     <sensor
       name="${link_name}_sensor"
@@ -53,14 +53,10 @@
       downsample:=1
       noise_mean:=0.0
-      noise_stddev:=0.01">
+      noise_stddev:=0.0">
     <link name="${link_name}">
       <pose>${link_pose}</pose>
-      <inertial>
-        <mass>0.1</mass>
-        <inertia>
-          <ixx>0.000166667</ixx>
-          <iyy>0.000166667</iyy>
-          <izz>0.000166667</izz>
-        </inertia>
+      <!-- Body envelope (x/y/z): 105 x 131.6 x 65 mm; mass: 1120 g. -->
+      <inertial auto="true">
+        <mass>1.120</mass>
       </inertial>
       <xacro:if value="${mesh_file != ''}">
@@ -85,7 +81,8 @@
       </xacro:if>
       <collision name="${link_name}_collision">
+        <density>1246.979970</density>
         <geometry>
           <box>
-            <size>0.1 0.1 0.1</size>
+            <size>0.105 0.1316 0.065</size>
           </box>
         </geometry>

File: src/livox_lidar_gz_sensor/urdf/livox_avia.xacro (robot description, xacro)
@@ -17,5 +17,5 @@
       downsample:=1
       noise_mean:=0.0
-      noise_stddev:=0.01">
+      noise_stddev:=0.0">
     <sensor
       name="${link_name}_sensor"
@@ -53,14 +53,10 @@
       downsample:=1
       noise_mean:=0.0
-      noise_stddev:=0.01">
+      noise_stddev:=0.0">
     <link name="${link_name}">
       <pose>${link_pose}</pose>
-      <inertial>
-        <mass>0.1</mass>
-        <inertia>
-          <ixx>0.000166667</ixx>
-          <iyy>0.000166667</iyy>
-          <izz>0.000166667</izz>
-        </inertia>
+      <!-- Body envelope (x/y/z): 91 x 61.2 x 64.8 mm; mass: 498 g. -->
+      <inertial auto="true">
+        <mass>0.498</mass>
       </inertial>
       <xacro:if value="${mesh_file != ''}">
@@ -85,7 +81,8 @@
       </xacro:if>
       <collision name="${link_name}_collision">
+        <density>1379.944190</density>
         <geometry>
           <box>
-            <size>0.1 0.1 0.1</size>
+            <size>0.091 0.0612 0.0648</size>
           </box>
         </geometry>

File: src/livox_lidar_gz_sensor/urdf/livox_horizon.xacro (robot description, xacro)
@@ -17,5 +17,5 @@
       downsample:=1
       noise_mean:=0.0
-      noise_stddev:=0.01">
+      noise_stddev:=0.0">
     <sensor
       name="${link_name}_sensor"
@@ -44,5 +44,5 @@
       link_pose:='0 0 0 0 0 0'
       sensor_pose:='0 0 0 0 0 0'
-      mesh_file:='$(find livox_lidar_gz_sensor)/meshes/horizon.dae'
+      mesh_file:=''
       mesh_scale:='1 1 1'
       mesh_pose:='0 0 0 0 0 0'
@@ -53,7 +53,8 @@
       downsample:=1
       noise_mean:=0.0
-      noise_stddev:=0.01">
+      noise_stddev:=0.0">
     <link name="${link_name}">
       <pose>${link_pose}</pose>
+      <!-- Placeholder dynamics only; Horizon mass and inertia are unverified. -->
       <inertial>
         <mass>0.1</mass>
@@ -75,13 +76,5 @@
         </visual>
       </xacro:if>
-      <xacro:if value="${mesh_file == ''}">
-        <visual name="${link_name}_visual_placeholder">
-          <geometry>
-            <box>
-              <size>0.1 0.1 0.1</size>
-            </box>
-          </geometry>
-        </visual>
-      </xacro:if>
+      <!-- Placeholder collision only; dimensions and point-cloud behavior are unverified. -->
       <collision name="${link_name}_collision">
         <geometry>

File: src/livox_lidar_gz_sensor/urdf/livox_mid360.xacro (robot description, xacro)
@@ -17,5 +17,5 @@
       downsample:=1
       noise_mean:=0.0
-      noise_stddev:=0.01">
+      noise_stddev:=0.0">
     <sensor
       name="${link_name}_sensor"
@@ -53,14 +53,10 @@
       downsample:=1
       noise_mean:=0.0
-      noise_stddev:=0.01">
+      noise_stddev:=0.0">
     <link name="${link_name}">
       <pose>${link_pose}</pose>
-      <inertial>
-        <mass>0.1</mass>
-        <inertia>
-          <ixx>0.000166667</ixx>
-          <iyy>0.000166667</iyy>
-          <izz>0.000166667</izz>
-        </inertia>
+      <!-- Body envelope (x/y/z): 65 x 65 x 60 mm; mass: 265 g. -->
+      <inertial auto="true">
+        <mass>0.265</mass>
       </inertial>
       <xacro:if value="${mesh_file != ''}">
@@ -85,7 +81,8 @@
       </xacro:if>
       <collision name="${link_name}_collision">
+        <density>1045.364892</density>
         <geometry>
           <box>
-            <size>0.1 0.1 0.1</size>
+            <size>0.065 0.065 0.060</size>
           </box>
         </geometry>

File: src/livox_lidar_gz_sensor/urdf/livox_mid40.xacro (robot description, xacro)
@@ -17,5 +17,5 @@
       downsample:=1
       noise_mean:=0.0
-      noise_stddev:=0.01">
+      noise_stddev:=0.0">
     <sensor
       name="${link_name}_sensor"
@@ -44,5 +44,5 @@
       link_pose:='0 0 0 0 0 0'
       sensor_pose:='0 0 0 0 0 0'
-      mesh_file:='$(find livox_lidar_gz_sensor)/meshes/mid40.dae'
+      mesh_file:=''
       mesh_scale:='1 1 1'
       mesh_pose:='0 0 0 0 0 0'
@@ -53,7 +53,8 @@
       downsample:=1
       noise_mean:=0.0
-      noise_stddev:=0.01">
+      noise_stddev:=0.0">
     <link name="${link_name}">
       <pose>${link_pose}</pose>
+      <!-- Placeholder dynamics only; Mid-40 mass and inertia are unverified. -->
       <inertial>
         <mass>0.1</mass>
@@ -75,13 +76,5 @@
         </visual>
       </xacro:if>
-      <xacro:if value="${mesh_file == ''}">
-        <visual name="${link_name}_visual_placeholder">
-          <geometry>
-            <box>
-              <size>0.1 0.1 0.1</size>
-            </box>
-          </geometry>
-        </visual>
-      </xacro:if>
+      <!-- Placeholder collision only; dimensions and point-cloud behavior are unverified. -->
       <collision name="${link_name}_collision">
         <geometry>

File: src/livox_lidar_gz_sensor/urdf/livox_mid70.xacro (robot description, xacro)
@@ -17,5 +17,5 @@
       downsample:=1
       noise_mean:=0.0
-      noise_stddev:=0.01">
+      noise_stddev:=0.0">
     <sensor
       name="${link_name}_sensor"
@@ -53,14 +53,10 @@
       downsample:=1
       noise_mean:=0.0
-      noise_stddev:=0.01">
+      noise_stddev:=0.0">
     <link name="${link_name}">
       <pose>${link_pose}</pose>
-      <inertial>
-        <mass>0.1</mass>
-        <inertia>
-          <ixx>0.000166667</ixx>
-          <iyy>0.000166667</iyy>
-          <izz>0.000166667</izz>
-        </inertia>
+      <!-- Body envelope (x/y/z): 97 x 64 x 62.7 mm; mass: 580 g. -->
+      <inertial auto="true">
+        <mass>0.58</mass>
       </inertial>
       <xacro:if value="${mesh_file != ''}">
@@ -85,7 +81,11 @@
       </xacro:if>
       <collision name="${link_name}_collision">
+        <!-- 0.58 kg / (0.097 m * 0.064 m * 0.0627 m). This keeps the
+             computed mass correct on SDFormat versions where density is used
+             when expanding auto inertia. -->
+        <density>1490.077114</density>
         <geometry>
           <box>
-            <size>0.1 0.1 0.1</size>
+            <size>0.097 0.064 0.0627</size>
           </box>
         </geometry>

File: src/livox_lidar_gz_sensor/urdf/livox_tele.xacro (robot description, xacro)
@@ -17,5 +17,5 @@
       downsample:=1
       noise_mean:=0.0
-      noise_stddev:=0.01">
+      noise_stddev:=0.0">
     <sensor
       name="${link_name}_sensor"
@@ -53,14 +53,10 @@
       downsample:=1
       noise_mean:=0.0
-      noise_stddev:=0.01">
+      noise_stddev:=0.0">
     <link name="${link_name}">
       <pose>${link_pose}</pose>
-      <inertial>
-        <mass>0.1</mass>
-        <inertia>
-          <ixx>0.000166667</ixx>
-          <iyy>0.000166667</iyy>
-          <izz>0.000166667</izz>
-        </inertia>
+      <!-- Body envelope (x/y/z): 122 x 112 x 94.2 mm; mass: 1800 g. -->
+      <inertial auto="true">
+        <mass>1.800</mass>
       </inertial>
       <xacro:if value="${mesh_file != ''}">
@@ -85,7 +81,8 @@
       </xacro:if>
       <collision name="${link_name}_collision">
+        <density>1398.439714</density>
         <geometry>
           <box>
-            <size>0.1 0.1 0.1</size>
+            <size>0.122 0.112 0.0942</size>
           </box>
         </geometry>
